File: cit_logo.kicad_pcb (KiCad board)
At the start: 2 copper layers, 49.8 x 67.4 mm, 19 parts, among them J1 Conn_01x02, J2 Conn_01x02

Commit message: Add files via upload
Parts:
- D1, D10, D11, D12, D13, D2, D3, D4, D5, D6, D7, D8, D9: footprint LED_SMD:LED_0402_1005Metric_Pad0.77x0.64mm_HandSolder -> LED_SMD:LED_0603_1608Metric_Pad1.05x0.95mm_HandSolder
- moved D3 0.15 mm to (144.9, 108.0)
Routing:
- net +3V3: track 70.9 -> 71.7 mm
- net GND: track 108.3 -> 107.7 mm
