File: cit_logo.kicad_pcb (KiCad board)
At the start: 2 copper layers, 49.8 x 67.4 mm, 19 parts, among them J1 Conn_01x02, J2 Conn_01x02

Commit message: Add files via upload
Parts:
- moved J1 0.45 mm to (153.1, 81.4)
Routing:
- net Net-(J1-Pad2): track 15.6 -> 22.1 mm
Changed lines of the file:
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@@
   )
   (footprint "Battery:BatteryHolder_Keystone_3034_1x20mm" (layer "B.Cu")
-    (at 152.654 81.407)
+    (at 153.1 81.4)
     (descr "Keystone 3034 SMD battery holder for 2020, 2025 and 2032 coincell batteries. http://www.keyelco.com/product-pdf.cfm?p=798")
     (tags "Keystone type 3034 coin cell retainer")
@@
     (fp_line (start -10.78 5.46) (end -10.78 3) (layer "B.SilkS") (width 0.12))
     (fp_line (start -8.7 7.54) (end -10.78 5.46) (layer "B.SilkS") (width 0.12))
+    (fp_line (start 10.78 -3.63) (end 9.34 -7.58) (layer "B.SilkS") (width 0.12))
     (fp_line (start -10.78 -3.63) (end -9.34 -7.58) (layer "B.SilkS") (width 0.12))
     (fp_line (start 10.78 5.46) (end 10.78 3) (layer "B.SilkS") (width 0.12))
-    (fp_line (start 10.78 -3.63) (end 9.34 -7.58) (layer "B.SilkS") (width 0.12))
     (fp_line (start -10.78 -3) (end -10.78 -3.63) (layer "B.SilkS") (width 0.12))
+    (fp_arc (start -9.34 -7.58) (mid -7.921654 -8.918739) (end -6.003354 -8.56653) (layer "B.SilkS") (width 0.12))
     (fp_arc (start 6 -8.55) (mid 7.90634 -8.911669) (end 9.325243 -7.588169) (layer "B.SilkS") (width 0.12))
-    (fp_arc (start -9.34 -7.58) (mid -7.921654 -8.918739) (end -6.003354 -8.56653) (layer "B.SilkS") (width 0.12))
     (fp_circle (center 0 0) (end 0 -10.25) (layer "Dwgs.User") (width 0.15) (fill none))
     (fp_line (start -11.87 -2.79) (end -10.88 -2.79) (layer "B.CrtYd") (width 0.05))
@@
   (via (at 147.3 111.8) (size 0.8) (drill 0.4) (layers "F.Cu" "B.Cu") (free) (net 0))
   (via (at 165.2 111.8) (size 0.8) (drill 0.4) (layers "F.Cu" "B.Cu") (free) (net 0))
-  (segment (start 141.669 81.407) (end 138.938 81.407) (width 0.45) (layer "B.Cu") (net 1))
   (segment (start 163.8785 103.8235) (end 163.816 103.886) (width 0.45) (layer "B.Cu") (net 1))
+  (segment (start 164.085 96.902) (end 164.719 97.536) (width 0.45) (layer "B.Cu") (net 1))
   (segment (start 144.4615 108.077) (end 144.79948 107.73902) (width 0.45) (layer "B.Cu") (net 1))
   (segment (start 160.02 105.3455) (end 160.147 105.4725) (width 0.45) (layer "B.Cu") (net 1))
   (segment (start 158.8915 102.7915) (end 160.02 102.7915) (width 0.45) (layer "B.Cu") (net 1))
+  (segment (start 135.128 95.0585) (end 135.128 85.217) (width 0.45) (layer "B.Cu") (net 1))
   (segment (start 144.79948 107.73902) (end 144.79948 104.18502) (width 0.45) (layer "B.Cu") (net 1))
-  (segment (start 163.576 99.695) (end 163.068 99.187) (width 0.45) (layer "B.Cu") (net 1))
   (segment (start 150.241 103.6945) (end 150.241 100.203) (width 0.45) (layer "B.Cu") (net 1))
-  (segment (start 135.128 95.0585) (end 141.859 101.7895) (width 0.45) (layer "B.Cu") (net 1))
   (segment (start 157.706 105.17) (end 160.147 105.17) (width 0.45) (layer "B.Cu") (net 1))
+  (segment (start 154.913 99.187) (end 154.672 99.428) (width 0.45) (layer "B.Cu") (net 1))
   (segment (start 154.672 108.204) (end 157.706 105.17) (width 0.45) (layer "B.Cu") (net 1))
   (segment (start 160.02 102.489) (end 160.02 105.3455) (width 0.45) (layer "B.Cu") (net 1))
-  (segment (start 163.639 81.407) (end 163.639 96.456) (width 0.45) (layer "B.Cu") (net 1))
   (segment (start 154.385 99.441) (end 154.672 99.728) (width 0.45) (layer "B.Cu") (net 1))
   (segment (start 141.859 106.934) (end 143.002 108.077) (width 0.45) (layer "B.Cu") (net 1))
-  (segment (start 138.938 81.407) (end 135.128 85.217) (width 0.45) (layer "B.Cu") (net 1))
-  (segment (start 164.719 100.076) (end 164.338 100.457) (width 0.45) (layer "B.Cu") (net 1))
-  (segment (start 163.068 99.187) (end 154.913 99.187) (width 0.45) (layer "B.Cu") (net 1))
+  (segment (start 164.719 97.536) (end 164.719 100.076) (width 0.45) (layer "B.Cu") (net 1))
+  (segment (start 141.859 101.7895) (end 135.128 95.0585) (width 0.45) (layer "B.Cu") (net 1))
+  (segment (start 163.576 99.695) (end 163.068 99.187) (width 0.45) (layer "B.Cu") (net 1))
   (segment (start 163.576 103.8235) (end 163.5135 103.886) (width 0.45) (layer "B.Cu") (net 1))
-  (segment (start 163.639 96.456) (end 164.719 97.536) (width 0.45) (layer "B.Cu") (net 1))
+  (segment (start 154.672 99.428) (end 154.672 99.728) (width 0.45) (layer "B.Cu") (net 1))
   (segment (start 158.623 102.523) (end 158.8915 102.7915) (width 0.45) (layer "B.Cu") (net 1))
-  (segment (start 164.338 100.457) (end 163.576 100.457) (width 0.45) (layer "B.Cu") (net 1))
+  (segment (start 164.085 81.4) (end 164.085 96.902) (width 0.45) (layer "B.Cu") (net 1))
   (segment (start 158.623 102.489) (end 158.623 102.523) (width 0.45) (layer "B.Cu") (net 1))
   (segment (start 144.79948 104.18502) (end 145.0985 103.886) (width 0.45) (layer "B.Cu") (net 1))
-  (segment (start 154.913 99.187) (end 154.672 99.428) (width 0.45) (layer "B.Cu") (net 1))
-  (segment (start 164.719 97.536) (end 164.719 100.076) (width 0.45) (layer "B.Cu") (net 1))
-  (segment (start 135.128 85.217) (end 135.128 95.0585) (width 0.45) (layer "B.Cu") (net 1))
   (segment (start 163.816 107.95) (end 163.943 108.077) (width 0.45) (layer "B.Cu") (net 1))
-  (segment (start 163.576 100.457) (end 163.576 99.695) (width 0.45) (layer "B.Cu") (net 1))
   (segment (start 154.3695 100.457) (end 156.591 100.457) (width 0.45) (layer "B.Cu") (net 1))
+  (segment (start 164.719 100.076) (end 164.338 100.457) (width 0.45) (layer "B.Cu") (net 1))
   (segment (start 154.672 99.728) (end 154.672 100.457) (width 0.45) (layer "B.Cu") (net 1))
   (segment (start 151.003 99.441) (end 154.385 99.441) (width 0.45) (layer "B.Cu") (net 1))
+  (segment (start 138.938 81.407) (end 142.108 81.407) (width 0.45) (layer "B.Cu") (net 1))
+  (segment (start 163.576 100.457) (end 163.576 99.695) (width 0.45) (layer "B.Cu") (net 1))
+  (segment (start 135.128 85.217) (end 138.938 81.407) (width 0.45) (layer "B.Cu") (net 1))
   (segment (start 150.0495 103.886) (end 150.241 103.6945) (width 0.45) (layer "B.Cu") (net 1))
   (segment (start 145.0985 100.457) (end 145.0985 100.521136) (width 0.45) (layer "B.Cu") (net 1))
+  (segment (start 163.068 99.187) (end 154.913 99.187) (width 0.45) (layer "B.Cu") (net 1))
   (segment (start 143.002 108.077) (end 144.4615 108.077) (width 0.45) (layer "B.Cu") (net 1))
   (segment (start 156.591 100.457) (end 158.623 102.489) (width 0.45) (layer "B.Cu") (net 1))
-  (segment (start 154.672 99.428) (end 154.672 99.728) (width 0.45) (layer "B.Cu") (net 1))
   (segment (start 145.401 103.886) (end 145.401 100.457) (width 0.45) (layer "B.Cu") (net 1))
+  (segment (start 142.108 81.407) (end 142.115 81.4) (width 0.45) (layer "B.Cu") (net 1))
+  (segment (start 164.338 100.457) (end 163.576 100.457) (width 0.45) (layer "B.Cu") (net 1))
   (segment (start 150.241 100.203) (end 151.003 99.441) (width 0.45) (layer "B.Cu") (net 1))
   (segment (start 145.0985 103.886) (end 150.0495 103.886) (width 0.45) (layer "B.Cu") (net 1))
@@
   (segment (start 145.909 108.891) (end 145.453 109.347) (width 0.45) (layer "B.Cu") (net 2))
   (segment (start 142.6135 105.4865) (end 141.859 105.4865) (width 0.45) (layer "B.Cu") (net 2))
-  (segment (start 157.405 95) (end 157.405 86.158) (width 0.45) (layer "B.Cu") (net 3))
+  (segment (start 157.405 85.705) (end 153.1 81.4) (width 0.45) (layer "B.Cu") (net 3))
+  (segment (start 157.405 95) (end 157.405 85.705) (width 0.45) (layer "B.Cu") (net 3))
   (segment (start 157.405 86.158) (end 152.654 81.407) (width 0.45) (layer "B.Cu") (net 3))
   (zone (net 0) (net_name "") (layer "F.Cu") (hatch edge 0.508)

Commit message: Add files via upload
Parts:
- added REF**: MountingHole_2.2mm_M2_DIN965, MountingHole:MountingHole_2.2mm_M2_DIN965, F.Cu at (152.8, 58.5)
- added X1: Badgelife_shitty_connector, cit:Badgelife-Shitty-2x2, F.Cu at (170.8, 89.1)
- added X2: Badgelife_shitty_connector, cit:Badgelife-Shitty-2x2, F.Cu at (135.3, 88.9)
Routing:
- net +3V3: track 71.7 -> 157.3 mm
- net GND: track 108.0 -> 89.6 mm
